File: Hardware/ADUM3160_USB_Isolator.kicad_pcb (KiCad board)
At the start: 2 copper layers, 55.9 x 20.3 mm, 24 parts, among them J1 USB-AM-S-X-X-TH, J2 USB_A, J3 Conn_01x03_Pin, J4 Conn_01x03_Pin, U1 ADUM3160

Commit message: Cleanup & Repo maintain
Routing:
- net GND: vias 13 -> 15
Changed lines of the file:
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@@
 		(tags "capacitor handsolder")
 		(property "Reference" "C5"
-			(at 0 -1.43 360)
+			(at 0 -1.43 0)
 			(layer "F.SilkS")
 			(effects
@@
 		)
 		(property "Value" "100n"
-			(at 0 1.43 360)
+			(at 0 1.43 0)
 			(layer "F.Fab")
 			(effects
@@
 		)
 		(fp_text user "${REFERENCE}"
-			(at 0 0 360)
+			(at 0 0 0)
 			(layer "F.Fab")
 			(effects
@@
 	)
 	(via
+		(at 116.332 87.757)
+		(size 0.6)
+		(drill 0.3)
+		(layers "F.Cu" "B.Cu")
+		(free yes)
+		(net 2)
+	)
+	(via
 		(at 124.079 99.187)
 		(size 0.6)
@@
 		(net 2)
 	)
+	(via
+		(at 116.586 91.059)
+		(size 0.6)
+		(drill 0.3)
+		(layers "F.Cu" "B.Cu")
+		(free yes)
+		(net 2)
+	)
